File: wattbreaker.kicad_pcb (KiCad board)
At the start: 2 copper layers, 47.4 x 34.1 mm, 33 parts, among them J1 Stomp, J2 Power, U1 TL072

Commit message: v0.1: initial revision
Other:
- board text added: "${FONT:gothitt}Wattbreaker"
- board text added: "${REVISION} ${DATE}"
- board text added: "${URL}"
- board text removed: "Wattbreaker"
Changed lines of the file:
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@@
     (pcbplotparams
       (layerselection 0x00010fc_ffffffff)
-      (disableapertmacros false)
-      (usegerberextensions false)
-      (usegerberattributes true)
+      (disableapertmacros true)
+      (usegerberextensions true)
+      (usegerberattributes false)
       (usegerberadvancedattributes true)
       (creategerberjobfile true)
@@
       (viasonmask false)
       (mode 1)
-      (useauxorigin false)
+      (useauxorigin true)
       (hpglpennumber 1)
       (hpglpenspeed 20)
@@
       (plotinvisibletext false)
       (sketchpadsonfab false)
-      (subtractmaskfromsilk false)
+      (subtractmaskfromsilk true)
       (outputformat 1)
       (mirror false)
-      (drillshape 1)
+      (drillshape 0)
       (scaleselection 1)
-      (outputdirectory "")
-    )
-  )
-  (property "DATE" "2021-01-06")
+      (outputdirectory "Gerber/")
+    )
+  )
+  (property "DATE" "2021-01-08")
   (property "REVISION" "v0.1")
   (property "TITLE" "Wattbreaker")
@@
   )
   (gr_rect (start 85.32 50.23) (end 132.72 84.325) (layer "Edge.Cuts") (width 0.1) (fill none))
-  (gr_text "Wattbreaker" (at 122.41 82.69) (layer "B.SilkS")
-    (effects (font (size 1.3 1.5) (thickness 0.2)) (justify mirror))
+  (gr_text "${REVISION}\n${DATE}" (at 131.02 76.65 90) (layer "B.SilkS")
+    (effects (font (size 0.8 0.8) (thickness 0.127)) (justify mirror))
+  )
+  (gr_text "${FONT:gothitt}Wattbreaker" (at 122.7 82.69) (layer "B.SilkS")
+    (effects (font (size 1.6 2.1) (thickness 0.15)) (justify mirror))
+  )
+  (gr_text "${URL}" (at 122.41 73.12 90) (layer "B.SilkS")
+    (effects (font (size 0.8 0.7) (thickness 0.127)) (justify mirror))
   )
   (segment (start 107.85 64.95) (end 109.72 63.08) (width 0.35) (layer "F.Cu") (net 1))

Commit message: updated to KiCad 6.0
Other:
- board text added: "Wattbreaker"
- board text removed: "${FONT:gothitt}Wattbreaker"
